Commit message: Squashed open source commit of KF Adaptive MPC paper
Gait sequencer updates

apply solver best MPC & WBC QP/solver settings

Hotfix: not initialized target when switching GAIT

Fixed zero values in foot_heights at beginning of a gait which eventually...

Pinnochio as main model

Merge branch 'kf_for_adaptive_mpc_paper' into 'main'

Kf for adaptive mpc paper

See merge request underactuated-robotics/quadruped-development/dfki-quad-ros2!228

Merge branch 'quick_readme_change' into 'main'

edited readme

See merge request underactuated-robotics/quadruped-development/dfki-quad-ros2!229

Hotfix Readme git tags

fix github actions be freeing disk space

File: ws/src/common/model/urdf/quad.urdf (robot description, URDF)
Before this commit: robot dfki-quad, 18 links, 17 joints
Links:
- added link link_belly_bottom
Joints:
- added joint joint_belly_bottom: type fixed, parent base_link, child link_belly_bottom, origin xyz=0 0 -0.06 rpy=0 0 0, axis 0 0 0
